File: _scheme/feeder-meteo-clock.sch (EAGLE design)
At the start: 8 parts, among them J1 RTC MH, M1 ARDUINO-PRO-MINI-5.0V, SW1 ExtraFeed

Commit message: ===DEVICE WWAS CREATED=== DONE: Created schematic and make some bugfixes
Parts:
- removed M1: ARDUINO-PRO-MINI-5.0V, diy-modules:ARDUINO-PRO-MINI-5.0V
- removed SV2: Button&leds, con-lstb:MA07-1
- removed SW1: ExtraFeed, special:SW_DIP-1
- added +3V1: +3V3(T), gm-supply:+18V(T)
- added EXTRA_FEED, EXTRA_FEED1, EXTRA_FEED2, EXTRA_FEED3: (no value), switch-omron:10-XX
- added LED1: (no value), led:LED3MM
- added M2: ARDUINO-NANO-3.0, diy-modules:ARDUINO-NANO-3.0
- added SERVO: (no value), pinhead:PINHD-1X3
Connections:
- new net +18V: +3V1.+18V, J1.VPP, M2.3V3, SERVO.1, U$1.VIN
- new net N$1: M2.A4, U$1.SDA
- new net N$13: J1.PGD, M2.D11/MOSI
- new net N$14: M2.D5, SV1.6
- new net N$15: M2.D6, SV1.5
- new net N$16: J1.GND, M2.D12/MISO
- new net N$17: LED1.A, M2.A6
- new net N$19: M2.A0, SERVO.3
- new net N$2: M2.A5, U$1.SCL
- new net N$20: EXTRA_FEED.S, EXTRA_FEED.S1, M2.D2
- new net N$21: M2.D7, SV1.4
- new net N$22: M2.D8, SV1.3
- new net N$23: M2.D9, SV1.2
- new net N$24: M2.D10, SV1.1
- new net N$3: EXTRA_FEED1.P, EXTRA_FEED1.P1, M2.A1
- new net N$4: J1.PGC, M2.D13/SCK
- new net N$5: EXTRA_FEED2.P, EXTRA_FEED2.P1, M2.A2
- new net N$6: EXTRA_FEED3.P, EXTRA_FEED3.P1, M2.A3
- net +9V: now also +9V1.+9V, M2.5V, SV1.10, SV1.8; no longer J1.VPP, M1.VCC, U$1.VIN
- net GND: now also EXTRA_FEED.P, EXTRA_FEED1.S, EXTRA_FEED2.S, EXTRA_FEED3.S, GND1.GND, LED1.C, M2.GND.2, SERVO.2, SV1.7, SV1.9
Other:
- moved on the sheet: J1, SV1, U$1
